File: libcsp-zephyr-hw.kicad_sch (KiCad schematic)
At the start: 31 parts, among them J1 NETWORK, J2 HARDWARE_ADDRESS, J3 JTAG+UART, J4 HC-05, U1 YAAJ_WeAct_BlackPill_Part_Lik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

Commit message: Add some resistor values
Parts:
- R5, R6: value R -> 4.7k
- R7, R8: value R -> 1k
Changed lines of the file:
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@@
     (in_bom yes) (on_board yes)
     (property "Reference" "R6" (id 0) (at 91.44 82.55 90))
-    (property "Value" "R" (id 1) (at 87.63 82.55 90)
-      (effects (font (size 1.27 1.27)) hide)
-    )
+    (property "Value" "4.7k" (id 1) (at 93.98 82.55 90))
     (property "Footprint" "Resistor_SMD:R_0805_2012Metric" (id 2) (at 93.218 82.55 90)
       (effects (font (size 1.27 1.27)) hide)
@@
     (in_bom yes) (on_board yes)
     (property "Reference" "R8" (id 0) (at 138.43 38.1 90))
-    (property "Value" "R" (id 1) (at 138.43 34.29 90)
-      (effects (font (size 1.27 1.27)) hide)
-    )
+    (property "Value" "1k" (id 1) (at 138.43 35.56 90))
     (property "Footprint" "Resistor_SMD:R_0805_2012Metric" (id 2) (at 138.43 39.878 90)
       (effects (font (size 1.27 1.27)) hide)
@@
   )
   (symbol (lib_id "Connector_Generic:Conn_02x03_Odd_Even") (at 125.73 38.1 0) (unit 1)
-    (in_bom yes) (on_board yes) (fields_autoplaced)
-    (property "Reference" "J2" (id 0) (at 127 29.21 0))
-    (property "Value" "HARDWARE_ADDRESS" (id 1) (at 127 31.75 0))
+    (in_bom yes) (on_board yes)
+    (property "Reference" "J2" (id 0) (at 127 26.67 0))
+    (property "Value" "HARDWARE_ADDRESS" (id 1) (at 127 29.21 0))
     (property "Footprint" "Connector_PinHeader_2.54mm:PinHeader_2x03_P2.54mm_Horizontal" (id 2) (at 125.73 38.1 0)
       (effects (font (size 1.27 1.27)) hide)
@@
   )
   (symbol (lib_id "power:+3.3V") (at 120.65 35.56 90) (unit 1)
-    (in_bom yes) (on_board yes) (fields_autoplaced)
+    (in_bom yes) (on_board yes)
     (property "Reference" "#PWR06" (id 0) (at 124.46 35.56 0)
       (effects (font (size 1.27 1.27)) hide)
     )
-    (property "Value" "+3.3V" (id 1) (at 116.84 35.5599 90)
+    (property "Value" "+3.3V" (id 1) (at 123.19 33.02 90)
       (effects (font (size 1.27 1.27)) (justify left))
     )
@@
   )
   (symbol (lib_id "power:+3.3V") (at 133.35 35.56 270) (unit 1)
-    (in_bom yes) (on_board yes) (fields_autoplaced)
+    (in_bom yes) (on_board yes)
     (property "Reference" "#PWR012" (id 0) (at 129.54 35.56 0)
       (effects (font (size 1.27 1.27)) hide)
     )
-    (property "Value" "+3.3V" (id 1) (at 137.16 35.5599 90)
+    (property "Value" "+3.3V" (id 1) (at 130.81 33.02 90)
       (effects (font (size 1.27 1.27)) (justify left))
     )
@@
     (in_bom yes) (on_board yes)
     (property "Reference" "R5" (id 0) (at 88.9 82.55 90))
-    (property "Value" "R" (id 1) (at 92.71 82.55 90)
-      (effects (font (size 1.27 1.27)) hide)
-    )
+    (property "Value" "4.7k" (id 1) (at 86.36 82.55 90))
     (property "Footprint" "Resistor_SMD:R_0805_2012Metric" (id 2) (at 87.122 82.55 90)
       (effects (font (size 1.27 1.27)) hide)
@@
     (in_bom yes) (on_board yes)
     (property "Reference" "R7" (id 0) (at 115.57 38.1 90))
-    (property "Value" "R" (id 1) (at 115.57 34.29 90)
-      (effects (font (size 1.27 1.27)) hide)
-    )
+    (property "Value" "1k" (id 1) (at 115.57 35.56 90))
     (property "Footprint" "Resistor_SMD:R_0805_2012Metric" (id 2) (at 115.57 39.878 90)
       (effects (font (size 1.27 1.27)) hide)
@@
     )
     (path "/c4bed6f6-ea7f-44ef-a3da-82590664200f"
-      (reference "R5") (unit 1) (value "R") (footprint "Resistor_SMD:R_0805_2012Metric")
+      (reference "R5") (unit 1) (value "4.7k") (footprint "Resistor_SMD:R_0805_2012Metric")
     )
     (path "/27d2bf98-a07d-40fc-8ac6-77a7ee1f1b2e"
-      (reference "R6") (unit 1) (value "R") (footprint "Resistor_SMD:R_0805_2012Metric")
+      (reference "R6") (unit 1) (value "4.7k") (footprint "Resistor_SMD:R_0805_2012Metric")
     )
     (path "/dfca46a5-03d7-4caa-af21-988acd354af4"
-      (reference "R7") (unit 1) (value "R") (footprint "Resistor_SMD:R_0805_2012Metric")
+      (reference "R7") (unit 1) (value "1k") (footprint "Resistor_SMD:R_0805_2012Metric")
     )
     (path "/7bd67683-da7a-40da-9af7-556a4d301a55"
-      (reference "R8") (unit 1) (value "R") (footprint "Resistor_SMD:R_0805_2012Metric")
+      (reference "R8") (unit 1) (value "1k") (footprint "Resistor_SMD:R_0805_2012Metric")
     )
     (path "/ce342ba5-3648-4e8c-abad-d4b281b5e17e"
